Commit message: fix a detached leg issue in the URDF and add v1 for the locomotion task

File: assets/yahboomcar_description/urdf/MUTO_fixed.urdf (robot description, URDF)
Before this commit: robot yahboomcar, 24 links, 23 joints
Joints:
- joint yz3_Joint: origin xyz=0.195684337632199 -0.0250512362876254 0.015861531236519 rpy=0 0 0 -> xyz=-0.049774060130825 -0.0504179449064464 0.0158615312365191

Commit message: fix rpy missing

File: assets/yahboomcar_description/urdf/MUTO_fixed.urdf (robot description, URDF)
Before this commit: robot yahboomcar, 24 links, 23 joints
Joints:
- joint yz3_Joint: origin xyz=-0.049774060130825 -0.0504179449064464 0.0158615312365191 -> xyz=-0.049774060130825 -0.0504179449064464 0.0158615312365191 rpy=0 0 0
